File: stm32-kicad/stm32-kicad-rev3.kicad_pcb (KiCad board)
At the start: 2 copper layers, 77.5 x 45.7 mm, 57 parts, among them P1 CONN_01X05, P10 CONN_01X05, P2 CONN_01X03, P3 CONN_01X03, P4 CONN_01X03, P41 CONN_01X03, P6 CONN_01X08, P7 CONN_01X03, P9 CONN_02X06, Q1 FDS6675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

Commit message: python camera viewer
Parts:
- turned RJ3 to 180 degrees
Connections:
- R6 pad 2: /STM32/M1B -> /STM32/M1B_0
- RJ3 pad 2: /STM32/M1B -> /STM32/M1B_0
- RJ4 pad 2: /STM32/M1A -> Net-(RJ4-Pad2)
- U2 pad 41: /STM32/M1A -> Net-(RJ4-Pad2)
- U2 pad 42: /STM32/M1B -> /STM32/M1B_0
Routing:
- net /STM32/M1B: track 40.1 -> 13.9 mm
- net /STM32/M1A: track 36.3 -> 15.0 mm
