File: stm32-kicad/stm32.sch (KiCad schematic (older format))
At the start: 39 parts, among them P1 CONN_01X05, P10 CONN_01X05, P4 CONN_01X03, P41 CONN_01X03, P6 CONN_01X08, P7 CONN_01X03, P9 CONN_02X06, SW1 SW_PUSH, SW2 SW_PUSH, U1 NCP1117ST18T3G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

Commit message: python camera viewer
Connections:
- net labels added: M1B_0
- wire segments 158 -> 154
